File: sch/arduino-wirewrap/arduino-wirewrap.sch (KiCad schematic (older format))
At the start: 2 parts, among them J1 Conn_02x34_Top_Bottom

Commit message: Connect VPP to 5V as standard says
Connections:
- net +5V: now also J1.18 (Pin_18), J1.52 (Pin_52)
Changed lines of the file:
@@
 Text HLabel 5950 3500 0    50   Input ~ 0
 PL7_D7
+$Comp
+L power:+5V #PWR?
+U 1 1 6004D8C5
+P 5950 4700
+F 0 "#PWR?" H 5950 4550 50  0001 C CNN
+F 1 "+5V" V 5965 4828 50  0000 L CNN
+F 2 "" H 5950 4700 50  0001 C CNN
+F 3 "" H 5950 4700 50  0001 C CNN
+	1    5950 4700
+	0    -1   -1   0
+$EndComp
+$Comp
+L power:+5V #PWR?
+U 1 1 6004DD98
+P 6450 4700
+F 0 "#PWR?" H 6450 4550 50  0001 C CNN
+F 1 "+5V" V 6465 4828 50  0000 L CNN
+F 2 "" H 6450 4700 50  0001 C CNN
+F 3 "" H 6450 4700 50  0001 C CNN
+	1    6450 4700
+	0    1    1    0
+$EndComp
 $EndSCHEMATC
